File: IR Remote/IR_Remote/IR_Remote.kicad_sch (KiCad schematic)
At the start: 0 parts

Commit message: Task 01, pcb done
dont forget about gitignore
Other:
- sheet RECEIVER: file TRANSMITTER.kicad_sch -> RECEIVER.kicad_sch
- company: (none) -> X
- title: (none) -> IR Remote
Changed lines of the file:
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@@
 	(generator_version "8.0")
 	(paper "A4")
+	(title_block
+		(title "IR Remote")
+		(date "2024-09-17")
+		(rev "v.1.0.0")
+		(company "X")
+		(comment 1 "X")
+		(comment 2 "X")
+		(comment 3 "IR Remote, School Project ")
+	)
 	(sheet
-		(at 53.34 71.12)
+		(at 85.09 78.74)
 		(size 59.69 30.48)
 		(stroke
@@
 		)
 		(property "Sheetname" "TRANSMITTER"
-			(at 60.96 88.9 0)
+			(at 114.935 93.98 0)
 			(effects
 				(font
@@
 					(color 0 0 0 1)
 				)
-				(justify left bottom)
 			)
 		)
 		(property "Sheetfile" "TRANSMITTER.kicad_sch"
-			(at 53.34 102.1846 0)
+			(at 85.09 109.8046 0)
+			(effects
+				(font
+					(size 1.27 1.27)
+				)
+				(justify left top)
+			)
+		)
+		(instances
+			(project "IR_Remote"
+				(path "/07d62ec6-6e59-42d0-a028-2e4cdf5deb8a"
+					(page "2")
+				)
+			)
+		)
+	)
+	(sheet
+		(at 156.21 78.74)
+		(size 59.69 30.48)
+		(stroke
+			(width 0.1524)
+			(type solid)
+			(color 0 0 0 1)
+		)
+		(fill
+			(color 255 255 255 1.0000)
+		)
+		(property "Sheetname" "RECEIVER"
+			(at 186.055 93.345 0)
+			(effects
+				(font
+					(face "Bahnschrift")
+					(size 5 5)
+					(color 0 0 0 1)
+				)
+			)
+		)
+		(property "Sheetfile" "RECEIVER.kicad_sch"
+			(at 156.21 109.8046 0)
 			(effects
 				(font
@@
 				)
 			)
-		)
-	)
-	(sheet
-		(at 134.62 77.47)
-		(size 59.69 30.48)
-		(stroke
-			(width 0.1524)
-			(type solid)
-			(color 0 0 0 1)
-		)
-		(fill
-			(color 255 255 255 1.0000)
-		)
-		(property "Sheetname" "RECEIVER"
-			(at 142.24 95.25 0)
-			(effects
-				(font
-					(face "Bahnschrift")
-					(size 5 5)
-					(color 0 0 0 1)
-				)
-				(justify left bottom)
-			)
-		)
-		(property "Sheetfile" "TRANSMITTER.kicad_sch"
-			(at 134.62 108.5346 0)
-			(effects
-				(font
-					(size 1.27 1.27)
-				)
-				(justify left top)
-			)
-		)
-		(instances
-			(project "IR_Remote"
-				(path "/07d62ec6-6e59-42d0-a028-2e4cdf5deb8a"
-					(page "2")
-				)
-			)
