File: Task01_fuk/Task01_fuk.kicad_pcb (KiCad board)
At the start: 2 copper layers, 21.3 x 26 mm, 28 parts, among them J1 Conn_01x02_Pin, J3 DC, J4 DC, Q1 BC547, U1 NE555P

Commit message: nothing
Routing:
- net GND: track 44.0 -> 96.5 mm
Other:
- board size 21.3 x 26 mm -> 20.3 x 26 mm
