File: TEST01_KiCAD/TEST01_KiCAD.kicad_sch (KiCad schematic)
At the start: 28 parts, among them J1 Conn_01x02_Pin, J3 DC, J4 DC, Q1 BC547, U1 NE555P

Commit message: test n125 - KiCAD
Parts:
- removed C1: 10uF/50V, Capacitor_THT:CP_Radial_D6.3mm_P2.50mm, symbol Device:C_Polarized
- removed C3: 100uF/16V, Capacitor_THT:CP_Radial_D6.3mm_P2.50mm, symbol Device:C_Polarized
- removed C4: 100pF, Capacitor_THT:C_Disc_D6.0mm_W2.5mm_P5.00mm, symbol Device:C
- removed C5: 100nF, Capacitor_THT:C_Disc_D6.0mm_W2.5mm_P5.00mm, symbol Device:C
- removed C6: 10nF, Capacitor_THT:C_Disc_D6.0mm_W2.5mm_P5.00mm, symbol Device:C
- removed D1: 1N4148, Diode_THT:D_DO-35_SOD27_P7.62mm_Horizontal, symbol Diode:1N4148
- removed D5: 1N4007, Diode_THT:D_DO-41_SOD81_P10.16mm_Horizontal, symbol Diode:1N4007
- removed D7, D8: LED, LED_THT:LED_D5.0mm_Clear, symbol Device:LED
- removed J4: DC, Connector_PinHeader_2.54mm:PinHeader_1x01_P2.54mm_Vertical, symbol Connector:Conn_01x01_Pin
- removed R8: 1.5k, Resistor_THT:R_Axial_DIN0207_L6.3mm_D2.5mm_P10.16mm_Horizontal, symbol Device:R
- removed R9: 1.1M, Resistor_THT:R_Axial_DIN0207_L6.3mm_D2.5mm_P10.16mm_Horizontal, symbol Device:R
- added C1: 100nF, Capacitor_THT:C_Disc_D6.0mm_W2.5mm_P5.00mm, symbol Device:C
- added C3: 10nF, Capacitor_THT:C_Disc_D6.0mm_W2.5mm_P5.00mm, symbol Device:C
- added D1: 1N4001, Diode_THT:D_DO-41_SOD81_P10.16mm_Horizontal, symbol Diode:1N4007
- added D5: R_LED, LED_THT:LED_D5.0mm_Clear, symbol Device:LED
- added IO1: NE555P, Package_DIP:DIP-8_W7.62mm, symbol Timer:NE555P
- added J2: DC, Connector_PinHeader_2.54mm:PinHeader_1x01_P2.54mm_Vertical, symbol Connector:Conn_01x01_Pin
- C2: value 1uF/50V -> 47uF/100V
- D2, D3, D4, D6: value 1N4007 -> 1N4001
- R1: value 22k -> 150R
- R2: value 15k -> 1k
- R3: value 2.7k -> 4.7k
- R4: value 220R -> 75k
- R5: value 470R -> 10k
- R6: value 150R -> 10k
- R7: value 680k -> 220k
- renumbered U1 to IO2, Q1 to T1
Connections:
- net BCE: now also IO2.3 (Q), R1.1; no longer T1.2 (B)
- net DIS: now also R4.2, R5.2, IO1.7 (DIS); no longer IO2.7 (DIS), R7.1
- net GND: now also D2.2 (A), T1.3 (E), C1.2, C3.2, D5.1 (K), IO1.1 (GND); no longer D4.2 (A), R3.1
- net TR: now also R7.1, C3.1; no longer R7.2
- net VCC: now also D4.1 (K), D1.1 (K), IO1.4 (R), IO1.8 (VCC); no longer D6.1 (K), R6.2
- net at J1.2 (Pin_2): now also D3.1 (K), D4.2 (A); no longer D4.1 (K)
- net LED_DIS: now reaches R2.1
- net LED_DIS: now also D6.2 (A), R6.2; no longer R1.1
- net at R6.1: now also IO2.7 (DIS), R7.2; no longer T1.1 (C)
- net THR: now reaches R4.1
- net THR: now also C2.1, IO1.2 (TR), IO1.6 (THR)
- net CV: now reaches IO2.5 (CV)
- net CV: now also R3.1
- removed net DC_OUT: C2.1, J3.1 (Pin_1), R1.2, R2.2, R3.2
- net VCCQ: no longer names the net of D2.1 (K)
- net VCCQ: now also J1.1 (Pin_1), D1.2 (A); no longer D6.2 (A)
- new net: IO1.3 (Q), R3.2
- new net: C1.1, IO1.5 (CV)
- new net: R1.2, T1.2 (B)
- new net: D5.2 (A), R2.2
- new net REP_NEG: J2.1 (Pin_1), T1.1 (C)
- new net REP_POS: D6.1 (K), J3.1 (Pin_1)
Other:
- note added: "AC 9V"
- note added: "REPRO OUT"
- note removed: "AC"
- note removed: "DC"
- company: (none) -> SPS NA PROSEKU, 3EA, L1
- title: TASK_01 -> TEST01_KiCAD
- moved on the sheet: IO2, T1
