File: KNOP/Task01/Task01.kicad_pcb (KiCad board)
At the start: 2 copper layers, 29 x 48 mm, 28 parts, among them J1 Conn_01x02_Pin, J3 DC, J4 DC, Q1 BC547, U1 NE555P

Commit message: folder changes
Parts:
- moved C6 4.15 mm to (176.0, 48.1), turned to 90 degrees
- moved J3 0.76 mm to (172.5, 44.3)
- moved J4 0.58 mm to (163.6, 44.3)
Routing:
- net GND: track 31.0 -> 26.7 mm
- net Net-(U1-CV): track 2.87 -> 4.92 mm
- net VCC: track 75.6 -> 74.0 mm
- net DC_OUT: track 20.6 -> 19.9 mm
Other:
- board text added: "Cesty: 0.5mm :3"
