File: KNOP/Task01/Task01.kicad_sch (KiCad schematic)
At the start: 28 parts, among them J1 Conn_01x02_Pin, J3 DC, J4 DC, Q1 BC547, U1 NE555P

Commit message: folder changes
Other:
- company: (none) -> SPS na Proseku
Changed lines of the file:
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@@
 		(date "2024-09-17")
 		(rev "v1.0.0")
+		(company "SPS na Proseku")
 		(comment 3 "Task 01, Uloha 01")
 	)
