File: KNOP/OptoCouplers/OptoCouplers.kicad_sch (KiCad schematic)
At the start: 10 parts

Commit message: Optocoupler update
Other:
- note added: "PS9121-F3-AX is 15Mb/S RS-485 speed is 10Mb/S"

Commit message: will be removed
Parts:
- added U1: VO2630, Package_DIP:DIP-8_W7.62mm, symbol Isolator:VO2630
Other:
- note added: "PS9121-F3-AX is 15Mb/s single ch"
- note added: "RS-485 max speed is 10Mb/s"
- note added: "TLP2270(TP4,E is 20Mb/s cost, for 10 units is 43,35CZK"
- note added: "VO0661T is 10Mb/s, cost for 10 units is 59,39CZK"
- note added: "VO2630 is 10Mb/s, cost for 10 units is 38,34CZK"
- note removed: "PS9121-F3-AX is 15Mb/S RS-485 speed is 10Mb/S"
Changed lines of the file:
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@@
 		)
 	)
-	(text "PS9121-F3-AX is 15Mb/S RS-485 speed is 10Mb/S"
-		(exclude_from_sim no)
-		(at 144.018 77.978 0)
+	(text "RS-485 max speed is 10Mb/s"
+		(exclude_from_sim no)
+		(at 168.656 68.58 0)
+		(effects
+			(font
+				(size 1.27 1.27)
+			)
+		)
+	)
+	(text "PS9121-F3-AX is 15Mb/s single ch"
+		(exclude_from_sim no)
+		(at 142.24 75.184 0)
+		(effects
+			(font
+				(size 1.27 1.27)
+			)
+		)
+	)
+	(text "TLP2270(TP4,E is 20Mb/s cost, for 10 units is 43,35CZK"
+		(exclude_from_sim no)
+		(at 143.764 86.614 0)
 		(effects
 			(font
@@
 		)
 	)
+	(text "VO0661T is 10Mb/s, cost for 10 units is 59,39CZK"
+		(exclude_from_sim no)
+		(at 140.97 83.82 0)
+		(effects
+			(font
+				(size 1.27 1.27)
+			)
+		)
+	)
 	(text "Vf = 1.2V\nIf = 20mA\nVcc = 3.3V (RPi)\n\nR = (Vcc - Vf) / If\nR = 105R ~ 110R\n\nIf [110R] = 19.09mA"
 		(exclude_from_sim no)
 		(at 231.14 64.77 0)
+		(effects
+			(font
+				(size 1.27 1.27)
+			)
+		)
+	)
+	(text "VO2630 is 10Mb/s, cost for 10 units is 38,34CZK"
+		(exclude_from_sim no)
+		(at 140.462 89.408 0)
 		(effects
 			(font
@@
 					(unit 1)
 				)
+			)
+		)
+	)
+	(symbol
+		(lib_id "Isolator:VO2630")
+		(at 85.09 83.82 0)
+		(unit 1)
+		(exclude_from_sim no)
+		(in_bom yes)
+		(on_board yes)
+		(dnp no)
+		(fields_autoplaced yes)
+		(property "Reference" "U1"
+			(at 88.1065 68.58 0)
+			(effects
+				(font
+					(size 1.27 1.27)
+				)
+				(justify left)
+			)
+		)
+		(property "Value" "VO2630"
+			(at 88.1065 71.12 0)
+			(effects
+				(font
+					(size 1.27 1.27)
+				)
+				(justify left)
+			)
+		)
+		(property "Footprint" "Package_DIP:DIP-8_W7.62mm"
+			(at 87.63 102.108 0)
+			(effects
+				(font
+					(size 1.27 1.27)
+				)
+				(hide yes)
+			)
+		)
+		(property "Datasheet" "https://www.vishay.com/doc?84732"
+			(at 74.93 74.93 0)
+			(effects
+				(font
+					(size 1.27 1.27)
+				)
+				(hide yes)
+			)
+		)
+		(property "Description" "Dual High Speed CMOS Compatible Optocoupler, dV/dt 1000/us, VCM 10, max 7V VCC, DIP-8"
+			(at 85.09 83.82 0)
+			(effects
+				(font
+					(size 1.27 1.27)
+				)
+				(hide yes)
+			)
+		)
+		(pin "8"
+		)
+		(pin "4"
+		)
+		(pin "1"
+		)
+		(pin "3"
+		)
+		(pin "5"
+		)
+		(pin "2"
+		)
+		(pin "6"
+		)
+		(pin "7"
+		)
+		(instances
+			(project ""
+				(path "/2d1c3ebc-b5b7-4bd6-ada4-e78c3f1503ff"
+					(reference "U1")
+					(unit 1)
+				)

Commit message: lil
Parts:
- added R1: 10k, symbol Device:R
- added U2: HCPL-0600, Package_SO:SOIC-8_3.9x4.9mm_P1.27mm, symbol Isolator:HCPL-0600
- added U4: 74LVC2G14, symbol 74xGxx:74LVC2G14
Connections:
- net +5V: now also U4.5 (VCC)
- net GND: now also U2.3 (C), U4.2 (GND)
- net GND_OUT: now also U2.5 (GND)
- new net: U2.2 (A), U4.6
- new net TX: U4.1
Other:
- note added: "1. Q: Do we need 5V or 3.3V? IO voltage of a RPi is 3.3V. 2. Q: Do we want the external power pin to be bi-directional? (both power input and power output). 3. Q: Are we using half-duplex RS-485 communication (2-wire) or full-duplex (4-wire) 4. Q: Do we want RS-485 to be bidiractional? 5. Q: []"
- note removed: "1. Q: Do we need 5V or 3.3V? IO voltage of a RPi is 3.3V. 2. Q: Do we want the external power pin to be bi-directional? (both power input and power output). 3. Q: [] 4. Q: [] 5. Q: []"
- moved on the sheet: U1
