File: KNOP/Police_lights/Police_lights.kicad_pcb (KiCad board)
At the start: 2 copper layers, 59.5 x 31.8 mm, 30 parts, among them J1 Conn_01x02_Pin, J2 DC, J3 DC, U1 NE555P, U2 NE555P

Commit message: Math-statistics
Parts:
- moved H1 20.8 mm to (226.2, 85.2)
- moved H2 12.1 mm to (140.5, 60.0)
Changed lines of the file:
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@@
 	(footprint "MountingHole:MountingHole_3.2mm_M3_DIN965_Pad_TopBottom"
 		(layer "F.Cu")
-		(at 152.5 58.25)
+		(at 140.5 60)
 		(descr "Mounting Hole 3.2mm, M3, DIN965")
 		(tags "mounting hole 3.2mm m3 din965")
@@
 	(footprint "MountingHole:MountingHole_3.2mm_M3_DIN965_Pad_TopBottom"
 		(layer "F.Cu")
-		(at 205.5 83.5)
+		(at 226.25 85.25)
 		(descr "Mounting Hole 3.2mm, M3, DIN965")
 		(tags "mounting hole 3.2mm m3 din965")
@@
 		)
 	)
+	(dimension
+		(type aligned)
+		(layer "F.Cu")
+		(pts
+			(xy 208.75 55.75) (xy 149.25 55.75)
+		)
+		(height 8.749999)
+		(gr_text "59.5000 mm"
+			(at 179 45.200001 0)
+			(layer "F.Cu")
+			(effects
+				(font
+					(size 1.5 1.5)
+					(thickness 0.3)
+				)
+			)
+		)
+		(format
+			(prefix "")
+			(suffix "")
+			(units 3)
+			(units_format 1)
+			(precision 4)
+		)
+		(style
+			(thickness 0.2)
+			(arrow_length 1.27)
+			(text_position_mode 0)
+			(extension_height 0.58642)
+			(extension_offset 0.5) keep_text_aligned)
+	)
+	(dimension
+		(type aligned)
+		(layer "F.Cu")
+		(pts
+			(xy 208 55) (xy 208 86.75)
+		)
+		(height -8.5)
+		(gr_text "31.7500 mm"
+			(at 214.7 70.875 90)
+			(layer "F.Cu")
+			(effects
+				(font
+					(size 1.5 1.5)
+					(thickness 0.3)
+				)
+			)
+		)
+		(format
+			(prefix "")
+			(suffix "")
+			(units 3)
+			(units_format 1)
+			(precision 4)
+		)
+		(style
+			(thickness 0.2)
+			(arrow_length 1.27)
+			(text_position_mode 0)
+			(extension_height 0.58642)
+			(extension_offset 0.5) keep_text_aligned)
+	)
 	(segment

Commit message: police lights plot
Parts:
- moved H1 20.8 mm to (205.5, 83.5)
- moved H2 12.1 mm to (152.5, 58.2)
- renumbered U1 to IO1, U2 to IO2
Connections:
- C6 pad 1: TR -> TR_2
- IO2 pad 6: TR -> TR_2
Routing:
- net TR_2: track 11.6 -> 35.9 mm
- net TR: track 15.6 -> 0.00 mm
