File: KNOP/Police_lights/Police_lights.kicad_sch (KiCad schematic)
At the start: 34 parts

Commit message: plotting + pcb
Parts:
- removed C?: 100uF/16V, Capacitor_THT:CP_Radial_D6.3mm_P2.50mm, symbol Device:C_Polarized
- removed C?: 10uF/50V, Capacitor_THT:CP_Radial_D6.3mm_P2.50mm, symbol Device:C_Polarized
- removed C?: 100nF, Capacitor_THT:C_Disc_D6.0mm_W2.5mm_P5.00mm, symbol Device:C
- removed C?: 1uF/50V, Capacitor_THT:CP_Radial_D6.3mm_P2.50mm, symbol Device:C_Polarized
- removed C?: 100pF, Capacitor_THT:C_Disc_D6.0mm_W2.5mm_P5.00mm, symbol Device:C
- removed D? (x4): LED, LED_THT:LED_D5.0mm_Clear, symbol Device:LED
- removed D?: W01G, Diode_THT:Diode_Bridge_Round_D9.8mm, symbol Diode_Bridge:W01G
- removed D? (x5): 1N4007, Diode_THT:D_DO-41_SOD81_P10.16mm_Horizontal, symbol Diode:1N4007
- removed J? (x2): DC, Connector_PinHeader_2.54mm:PinHeader_1x01_P2.54mm_Vertical, symbol Connector:Conn_01x01_Pin
- removed J?: Conn_01x02_Pin, Connector_PinHeader_2.54mm:PinHeader_1x02_P2.54mm_Vertical, symbol Connector:Conn_01x02_Pin
- removed R?: 15k, Resistor_THT:R_Axial_DIN0207_L6.3mm_D2.5mm_P10.16mm_Horizontal, symbol Device:R
- removed R?: 22k, Resistor_THT:R_Axial_DIN0207_L6.3mm_D2.5mm_P10.16mm_Horizontal, symbol Device:R
- removed R?: 2.7k, Resistor_THT:R_Axial_DIN0207_L6.3mm_D2.5mm_P10.16mm_Horizontal, symbol Device:R
- removed R?: 470R, Resistor_THT:R_Axial_DIN0207_L6.3mm_D2.5mm_P10.16mm_Horizontal, symbol Device:R
- removed R?: 1M, Resistor_THT:R_Axial_DIN0207_L6.3mm_D2.5mm_P10.16mm_Horizontal, symbol Device:R
- added C1, C4: 10uF/50V, Capacitor_THT:CP_Radial_D6.3mm_P2.50mm, symbol Device:C_Polarized
- added C2: 100pF, Capacitor_THT:C_Disc_D6.0mm_W2.5mm_P5.00mm, symbol Device:C
- added C6: 1uF/50V, Capacitor_THT:CP_Radial_D6.3mm_P2.50mm, symbol Device:C_Polarized
- added D6, D7, D8, D9: LED, LED_THT:LED_D5.0mm_Clear, symbol Device:LED
- added H1, H2: M3, MountingHole:MountingHole_3.2mm_M3_DIN965_Pad_TopBottom, symbol Mechanical:MountingHole_Pad
- added J2, J3: DC, Connector_PinHeader_2.54mm:PinHeader_1x01_P2.54mm_Vertical, symbol Connector:Conn_01x01_Pin
- added R1: 15k, Resistor_THT:R_Axial_DIN0207_L6.3mm_D2.5mm_P10.16mm_Horizontal, symbol Device:R
- added R2: 2.2k, Resistor_THT:R_Axial_DIN0207_L6.3mm_D2.5mm_P10.16mm_Horizontal, symbol Device:R
- added R3, R4: 10k, Resistor_THT:R_Axial_DIN0207_L6.3mm_D2.5mm_P10.16mm_Horizontal, symbol Device:R
- added R5: 100R, Resistor_THT:R_Axial_DIN0207_L6.3mm_D2.5mm_P10.16mm_Horizontal, symbol Device:R
- added R6: 1M, Resistor_THT:R_Axial_DIN0207_L6.3mm_D2.5mm_P10.16mm_Horizontal, symbol Device:R
- added R8: 470R, Resistor_THT:R_Axial_DIN0207_L6.3mm_D2.5mm_P10.16mm_Horizontal, symbol Device:R
- gave numbers to parts that had none: 11
Connections:
- net GND: now also C2.2, C4.2, C6.2, J3.1 (Pin_1), R2.1, R4.1
- net Q_1: now also R8.2; no longer IO2.3 (Q)
- net Q_2: now also IO2.3 (Q), D6.2 (A), D7.1 (K), R6.1
- net TR: now also C6.1; no longer C5.1, IO1.2 (TR), IO1.6 (THR), IO2.2 (TR), R7.2
- net at D1.1 (K): now also C1.1, R1.2, R3.2, R5.2
- new net: C1.2, C2.1
- new net: D6.1 (K), D7.2 (A), D8.2 (A), D9.1 (K)
- new net: C4.1, R5.1
- new net: D8.1 (K), D9.2 (A), R8.1
- new net: R3.1, R4.2
- new net DIVIDER: J2.1 (Pin_1), R1.1, R2.2
- new net TR_1: C5.1, IO1.2 (TR), IO1.6 (THR), R7.2
- new net TR_2: IO2.2 (TR), R6.2
- no-connect marks 6 -> 8
Other:
- note added: "VOLTAGE DIVIDER"
- note removed: "DC"
- moved on the sheet: C3, C5, D1, IO1, IO2, R7

Commit message: police lights plot
Connections:
- net TR is gone; now on net TR_2: C6.1, IO2.6 (THR)
Other:
- moved on the sheet: H1, H2
Changed lines of the file:
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@@
 (kicad_sch
-	(version 20231120)
+	(version 20250114)
 	(generator "eeschema")
-	(generator_version "8.0")
+	(generator_version "9.0")
 	(paper "A4")
+	(rectangle
+		(start 22.225 27.94)
+		(end 102.87 73.66)
+		(stroke
+			(width 0)
+			(type dash_dot)
+			(color 0 0 0 1)
+		)
+		(fill
+			(type none)
+		)
+	)
+	(rectangle
+		(start 107.315 27.94)
+		(end 187.96 73.66)
+		(stroke
+			(width 0)
+			(type dash_dot)
+			(color 0 0 0 1)
+		)
+		(fill
+			(type none)
+		)
+	)
+	(rectangle
+		(start 191.77 27.94)
+		(end 272.415 73.66)
+		(stroke
+			(width 0)
+			(type dash_dot)
+			(color 0 0 0 1)
+		)
+		(fill
+			(type none)
+		)
+	)
+	(rectangle
+		(start 107.315 80.01)
+		(end 187.96 125.73)
+		(stroke
+			(width 0)
+			(type dash_dot)
+			(color 0 0 0 1)
+		)
+		(fill
+			(type none)
+		)
+	)
+	(rectangle
+		(start 22.225 80.01)
+		(end 102.87 125.73)
+		(stroke
+			(width 0)
+			(type dash_dot)
+			(color 0 0 0 1)
+		)
+		(fill
+			(type none)
+		)
+	)
+	(text "VOLTAGE DIVIDER"
+		(exclude_from_sim no)
+		(at 92.71 95.885 0)
+		(effects
+			(font
+				(face "Bahnschrift")
+				(size 1.5 1.5)
+				(color 0 0 0 1)
+			)
+		)
+	)
+	(text "AC"
+		(exclude_from_sim no)
+		(at 29.21 52.705 0)
+		(effects
+			(font
+				(face "Bahnschrift")
+				(size 2 2)
+				(color 0 0 0 1)
+			)
+		)
+	)
 	(junction
 		(at 226.06 45.72)
@@
 	)
 	(no_connect
-		(at 76.2 121.92)
+		(at 93.98 67.31)
 	)
 	(no_connect
-		(at 66.04 121.92)
+		(at 83.82 67.31)
 	)
 	(no_connect
@@
 		)
 	)
-	(rectangle
-		(start 22.225 27.94)
-		(end 102.87 73.66)
-		(stroke
-			(width 0)
-			(type dash_dot)
-			(color 0 0 0 1)
-		)
-		(fill
-			(type none)
-		)
-	)
-	(rectangle
-		(start 107.315 27.94)
-		(end 187.96 73.66)
-		(stroke
-			(width 0)
-			(type dash_dot)
-			(color 0 0 0 1)
-		)
-		(fill
-			(type none)
-		)
-	)
-	(rectangle
-		(start 191.77 27.94)
-		(end 272.415 73.66)
-		(stroke
-			(width 0)
-			(type dash_dot)
-			(color 0 0 0 1)
-		)
-		(fill
-			(type none)
-		)
-	)
-	(rectangle
-		(start 107.315 80.01)
-		(end 187.96 125.73)
-		(stroke
-			(width 0)
-			(type dash_dot)
-			(color 0 0 0 1)
-		)
-		(fill
-			(type none)
-		)
-	)
-	(rectangle
-		(start 22.225 80.01)
-		(end 102.87 125.73)
-		(stroke
-			(width 0)
-			(type dash_dot)
-			(color 0 0 0 1)
-		)
-		(fill
-			(type none)
-		)
-	)
-	(text "VOLTAGE DIVIDER"
-		(exclude_from_sim no)
-		(at 92.71 95.885 0)
-		(effects
-			(font
-				(face "Bahnschrift")
-				(size 1.5 1.5)
-				(color 0 0 0 1)
-			)
-		)
-	)
-	(text "AC"
-		(exclude_from_sim no)
-		(at 29.21 52.705 0)
-		(effects
-			(font
-				(face "Bahnschrift")
-				(size 2 2)
-				(color 0 0 0 1)
-			)
-		)
-	)
 	(global_label "Q_2"
 		(shape input)
@@
 		)
 	)
-	(global_label "TR"
+	(global_label "TR_2"
 		(shape input)
 		(at 171.45 107.95 0)
@@
 		)
 		(property "Intersheetrefs" "${INTERSHEET_REFS}"
-			(at 175.2392 107.95 0)
+			(at 176.5708 107.95 0)
 			(effects
 				(font
@@
 	(symbol
 		(lib_id "Mechanical:MountingHole_Pad")
-		(at 66.04 119.38 0)
+		(at 83.82 64.77 0)
 		(unit 1)
-		(exclude_from_sim yes)
+		(exclude_from_sim no)
 		(in_bom no)
 		(on_board yes)
@@
 		(fields_autoplaced yes)
 		(property "Reference" "H1"
-			(at 68.58 116.8399 0)
+			(at 86.36 62.2299 0)
 			(effects
 				(font
@@
 		)
 		(property "Value" "M3"
-			(at 68.58 119.3799 0)
+			(at 86.36 64.7699 0)
 			(effects
 				(font
@@
 		)
 		(property "Footprint" "MountingHole:MountingHole_3.2mm_M3_DIN965_Pad_TopBottom"
-			(at 66.04 119.38 0)
+			(at 83.82 64.77 0)
 			(effects
 				(font
@@
 		)
 		(property "Datasheet" "~"
-			(at 66.04 119.38 0)
+			(at 83.82 64.77 0)
 			(effects
 				(font
@@
 		)
 		(property "Description" "Mounting Hole with connection"
-			(at 66.04 119.38 0)
+			(at 83.82 64.77 0)
 			(effects
 				(font
@@
 	(symbol
 		(lib_id "Mechanical:MountingHole_Pad")
-		(at 76.2 119.38 0)
+		(at 93.98 64.77 0)
 		(unit 1)
-		(exclude_from_sim yes)
+		(exclude_from_sim no)
 		(in_bom no)
 		(on_board yes)
@@
 		(fields_autoplaced yes)
 		(property "Reference" "H2"
-			(at 78.74 116.8399 0)
+			(at 96.52 62.2299 0)
 			(effects
 				(font
@@
 		)
 		(property "Value" "M3"
-			(at 78.74 119.3799 0)
+			(at 96.52 64.7699 0)
 			(effects
 				(font
@@
 		)
 		(property "Footprint" "MountingHole:MountingHole_3.2mm_M3_DIN965_Pad_TopBottom"
-			(at 76.2 119.38 0)
+			(at 93.98 64.77 0)
 			(effects
 				(font
@@
 		)
 		(property "Datasheet" "~"
-			(at 76.2 119.38 0)
+			(at 93.98 64.77 0)
 			(effects
 				(font
@@
 		)
 		(property "Description" "Mounting Hole with connection"
-			(at 76.2 119.38 0)
+			(at 93.98 64.77 0)
 			(effects
 				(font
@@
 		)
 	)
+	(embedded_fonts no)
 )
