File: LF_LAP_TIMER/LF_LAP_TIMER.kicad_pcb (KiCad board)
At the start: 2 copper layers, 13 parts, among them J1 LCD I2C EXPANDER, SW1 ARM, SW2 STOP, SW3 RESTART

Commit message: final version
Parts:
- removed R3: 10K, Resistor_THT:R_Axial_DIN0207_L6.3mm_D2.5mm_P10.16mm_Horizontal
- added H1: MountingHole_Pad, MountingHole:MountingHole_3.2mm_M3_Pad, F.Cu at (83.6, 103.6)
- added H2: MountingHole_Pad, MountingHole:MountingHole_3.2mm_M3_Pad, F.Cu at (170.9, 103.6)
- added H3: MountingHole_Pad, MountingHole:MountingHole_3.2mm_M3_Pad, F.Cu at (170.9, 46.2)
- added H4: MountingHole_Pad, MountingHole:MountingHole_3.2mm_M3_Pad, F.Cu at (83.6, 46.2)
- added J2: SENSOR TERMINAL, TerminalBlock:TerminalBlock_MaiXu_MX126-5.0-05P_1x05_P5.00mm, F.Cu at (169.9, 66.5)
- added J3: LCD TERMINAL, TerminalBlock:TerminalBlock_MaiXu_MX126-5.0-05P_1x05_P5.00mm, F.Cu at (122.7, 102.6)
- added R10: 10K, Resistor_THT:R_Axial_DIN0207_L6.3mm_D2.5mm_P10.16mm_Horizontal, F.Cu at (117.3, 92.2)
- added R8: 10k, Resistor_THT:R_Axial_DIN0207_L6.3mm_D2.5mm_P10.16mm_Horizontal, F.Cu at (142.1, 83.1)
- added R9: 10K, Resistor_THT:R_Axial_DIN0207_L6.3mm_D2.5mm_P10.16mm_Horizontal, F.Cu at (127.5, 89.2)
- A1: moved to F.Cu
- J1: value LCD I2C EXPANDER -> SENSOR TERMINAL; footprint Connector_PinSocket_2.54mm:PinSocket_1x04_P2.54mm_Vertical -> TerminalBlock:TerminalBlock_MaiXu_MX126-5.0-02P_1x02_P5.00mm
- R1, R2: value 10K -> 0R
- R4: value 1k -> 10K
- R5: value 10k -> 10K
- R7: value 10K -> 1k
- moved J1 74.1 mm to (170.0, 53.5), turned to -90 degrees
- moved SW1 68.0 mm to (161.0, 102.6), turned to 180 degrees
- moved R7 65.3 mm to (154.8, 89.0), turned to 90 degrees
- moved SW2 57.2 mm to (148.2, 102.6), turned to 180 degrees
- moved A1 52.2 mm to (124.3, 46.7)
- moved R2 51.2 mm to (151.6, 89.0), turned to 90 degrees
- moved SW3 49.7 mm to (135.8, 102.6), turned to 180 degrees
- moved R6 44.4 mm to (132.0, 92.2)
- moved R5 43.6 mm to (132.0, 89.2)
- moved R4 42.8 mm to (132.0, 86.1)
- moved C1 34.7 mm to (154.8, 91.9)
- moved R1 32.1 mm to (158.0, 89.0), turned to 90 degrees
Connections:
- A1 pad 18: ARM_D3 -> unconnected-(A1-D3-Pad18)
- A1 pad 19: STOP_D4 -> unconnected-(A1-D4-Pad19)
- A1 pad 20: RST_D5 -> ARM_D5
- A1 pad 21: unconnected-(A1-D6-Pad21) -> STOP_D6
- A1 pad 22: unconnected-(A1-D7-Pad22) -> RST_D7
- J1 pad 2: +5V -> +12V
- R1 pad 1: +5V -> RELAY_OUT
- R1 pad 2: ARM_D3 -> RELAY_OUT_NC
- R2 pad 1: +5V -> RELAY_OUT
- R2 pad 2: STOP_D4 -> RELAY_OUT_NO
- R4 pad 1: Net-(A1-D2) -> +5V
- R4 pad 2: RELAY_OUTPUT -> ARM_D5
- R5 pad 1: Net-(A1-D2) -> +5V
- R5 pad 2: +5V -> STOP_D6
- R6 pad 2: SDA -> RST_D7
- R7 pad 1: SCL -> Net-(A1-D2)
- R7 pad 2: +5V -> RELAY_OUT
- SW1 pad 2: ARM_D3 -> ARM_D5
- SW2 pad 2: STOP_D4 -> STOP_D6
- SW3 pad 2: RST_D5 -> RST_D7
Routing:
- net +5V: track 0.00 -> 87.2 mm
- net +12V: track 0.00 -> 40.8 mm
- net ARM_D5: track 0.00 -> 23.0 mm
- net Net-(A1-D2): track 0.00 -> 22.4 mm
- net RELAY_OUT_NO: track 0.00 -> 19.2 mm
- net RST_D7: track 0.00 -> 17.3 mm
- net RELAY_OUT_NC: track 0.00 -> 17.2 mm
- net RELAY_OUT: track 0.00 -> 16.0 mm
- net STOP_D6: track 0.00 -> 15.1 mm
- net SDA: track 0.00 -> 14.5 mm
- net SCL: track 0.00 -> 13.4 mm
- added copper zone on B.Cu, net GND
Other:
- board outline added: 94.5 x 64.5 mm
- board text added: "12V"
- board text added: "2.1mm BARREL JACK"
- board text added: "5V"
- board text added: "ARM"
- board text added: "COM"
- board text added: "GND"
- board text added: "LCD"
- board text added: "LINE FOLLOWER LAP TIMER"
- board text added: "MADE BY: Savva Popov"
- board text added: "NC"
- board text added: "NO"
- board text added: "RESET"
- board text added: "SCL"
- board text added: "SDA"
- board text added: "SENSOR - EMITTER"
- board text added: "SENSOR - RECIEVER"
- board text added: "STOP"
- board text added: "USB"

Commit message: Lap timer plots
Routing:
- net SDA: track 14.5 -> 15.1 mm
- net RELAY_OUT_NC: track 17.2 -> 16.6 mm
