File: charliesSDCard/charliesSd.kicad_pcb (KiCad board)
At the start: 2 copper layers, 12 parts

Commit message: pcb updates
(no update)
Parts:
- moved SD1 13.2 mm to (103.7, 108.6)
- moved MC1 9.49 mm to (122.7, 100.2), turned to 180 degrees
