File: Charlie-SD-CARD/Charlie-SD-CARD.kicad_sch (KiCad schematic)
At the start: 12 parts

Commit message: charlie sd card
Parts:
- C1, C2, C3: footprint footprints:capacitor1 -> Capacitor_SMD:C_0402_1005Metric
- MEM1, MEM2: footprint footprints:memory -> Package_SO:TSOP-I-48_18.4x12mm_P0.5mm
- R1, R2, R3, R4, R5: footprint footprints:resistor1 -> Resistor_SMD:R_0402_1005Metric
Other:
- moved on the sheet: C1, C2, C3, R1, R2, R3, R4, R5

Commit message: sd card final edit
Parts:
- C1, C2, C3: footprint Capacitor_SMD:C_0402_1005Metric -> Capacitor_SMD:C_0402_1005Metric_Pad0.74x0.62mm_HandSolder
- MC1: footprint footprints:mc -> gps-compass_brd:Rosie_is_a_stupid_little_bitch_but_I_love_her
- R1, R2, R3, R4, R5: footprint Resistor_SMD:R_0402_1005Metric -> Resistor_SMD:R_0402_1005Metric_Pad0.72x0.64mm_HandSolder
Changed lines of the file:
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@@
 			)
 		)
-		(property "Footprint" "Resistor_SMD:R_0402_1005Metric"
+		(property "Footprint" "Resistor_SMD:R_0402_1005Metric_Pad0.72x0.64mm_HandSolder"
 			(at 127 180.848 90)
 			(effects
@@
 			)
 		)
-		(property "Footprint" "Resistor_SMD:R_0402_1005Metric"
+		(property "Footprint" "Resistor_SMD:R_0402_1005Metric_Pad0.72x0.64mm_HandSolder"
 			(at 127 165.608 90)
 			(effects
@@
 			)
 		)
-		(property "Footprint" "Resistor_SMD:R_0402_1005Metric"
+		(property "Footprint" "Resistor_SMD:R_0402_1005Metric_Pad0.72x0.64mm_HandSolder"
 			(at 127 157.988 90)
 			(effects
@@
 			)
 		)
-		(property "Footprint" "Capacitor_SMD:C_0402_1005Metric"
+		(property "Footprint" "Capacitor_SMD:C_0402_1005Metric_Pad0.74x0.62mm_HandSolder"
 			(at 86.36 149.5552 0)
 			(effects
@@
 			)
 		)
-		(property "Footprint" "Capacitor_SMD:C_0402_1005Metric"
+		(property "Footprint" "Capacitor_SMD:C_0402_1005Metric_Pad0.74x0.62mm_HandSolder"
 			(at 86.36 164.7952 0)
 			(effects
@@
 			)
 		)
-		(property "Footprint" "Resistor_SMD:R_0402_1005Metric"
+		(property "Footprint" "Resistor_SMD:R_0402_1005Metric_Pad0.72x0.64mm_HandSolder"
 			(at 127 150.368 90)
 			(effects
@@
 			)
 		)
-		(property "Footprint" "footprints:mc"
+		(property "Footprint" "gps-compass_brd:Rosie_is_a_stupid_little_bitch_but_I_love_her"
 			(at 97.79 59.69 0)
 			(effects
@@
 			)
 		)
-		(property "Footprint" "Capacitor_SMD:C_0402_1005Metric"
+		(property "Footprint" "Capacitor_SMD:C_0402_1005Metric_Pad0.74x0.62mm_HandSolder"
 			(at 86.36 157.1752 0)
 			(effects
@@
 			)
 		)
-		(property "Footprint" "Resistor_SMD:R_0402_1005Metric"
+		(property "Footprint" "Resistor_SMD:R_0402_1005Metric_Pad0.72x0.64mm_HandSolder"
 			(at 127 173.228 90)
 			(effects

Commit message: charlie SD update
Parts:
- SD1: footprint footprints:sdCard -> sumec_brd:sd_card_contacts
Connections:
- net DAT2/X: now also SD1.9; no longer SD1.0
Changed lines of the file:
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@@
 			)
 		)
-		(property "Footprint" "footprints:sdCard"
+		(property "Footprint" "sumec_brd:sd_card_contacts"
 			(at 44.45 96.52 0)
 			(effects
@@
 		(pin "5"
 		)
-		(pin "0"
+		(pin "9"
 		)
 		(pin "1"
