File: surgery/surgery.kicad_pcb (KiCad board)
At the start: 2 copper layers, 17.2 x 21.8 mm, 4 parts, among them J1 Conn_01x05_Pin, U2 LM66100Q, U3 LM66100Q, U4 LM66100Q

Commit message: plotting
Parts:
- added C2: 1uF, Capacitor_Tantalum_SMD:CP_EIA-3216-18_Kemet-A, F.Cu at (155.5, 64.3)
- added C3: 1uF, Capacitor_Tantalum_SMD:CP_EIA-3216-18_Kemet-A, F.Cu at (155.5, 58.0)
- added C4: 1uF, Capacitor_Tantalum_SMD:CP_EIA-3216-18_Kemet-A, F.Cu at (155.5, 52.3)
- added R4: 10k, Resistor_SMD:R_0805_2012Metric, F.Cu at (147.2, 58.0)
- added R6: 10k, Resistor_SMD:R_0805_2012Metric, F.Cu at (147.2, 52.5)
- added TP1: TestPoint, TestPoint:TestPoint_Loop_D1.80mm_Drill1.0mm_Beaded, F.Cu at (147.2, 61.0)
- added TP2: TestPoint, TestPoint:TestPoint_Loop_D1.80mm_Drill1.0mm_Beaded, F.Cu at (147.2, 49.5)
- moved U3 37.6 mm to (155.5, 55.3), turned to 180 degrees
- moved U4 35.1 mm to (155.5, 49.5), turned to 180 degrees
- moved J1 34.9 mm to (161.5, 63.8)
- moved U2 33.1 mm to (155.5, 61.0), turned to 180 degrees
Connections:
- J1 pad 1: raw_5V -> GND
- J1 pad 2: USB_MAIN_Vbus -> SRC_5V
- J1 pad 3: brown-out -> VBUS
- J1 pad 4: supercap -> BRWN
- J1 pad 5: GND -> SUPERCAP
- U2 pad 1: raw_5V -> SRC_5V
- U2 pad 3: USB_MAIN_Vbus -> VBUS
- U2 pad 5: GND -> Net-(U2-ST)
- U2 pad 6: brown-out -> BRWN
- U3 pad 1: USB_MAIN_Vbus -> VBUS
- U3 pad 3: raw_5V -> Net-(U2-ST)
- U3 pad 5: GND -> unconnected-(U3-ST-Pad5)
- U3 pad 6: brown-out -> BRWN
- U4 pad 1: brown-out -> BRWN
- U4 pad 3: supercap -> SUPERCAP
- U4 pad 5: GND -> Net-(U4-ST)
- U4 pad 6: supercap -> SUPERCAP
Routing:
- net Net-(U2-ST): track 0.00 -> 29.3 mm, vias 0 -> 4
- net BRWN: track 0.00 -> 29.2 mm
- net SUPERCAP: track 0.00 -> 21.4 mm, vias 0 -> 2
- net USB_MAIN_Vbus: track 20.4 -> 0.00 mm, vias 4 -> 0
- net SRC_5V: track 0.00 -> 19.4 mm
- net brown-out: track 18.8 -> 0.00 mm
- net raw_5V: track 14.8 -> 0.00 mm, vias 2 -> 0
- net supercap: track 14.3 -> 0.00 mm
- net Net-(U4-ST): track 0.00 -> 10.3 mm
- net VBUS: track 0.00 -> 9.44 mm
- net GND: track 19.0 -> 13.0 mm
Other:
- board size 17.2 x 21.8 mm -> 21.5 x 20.8 mm
- board text added: "B/O"
- board text added: "IN1"
- board text added: "IN2"
- board text added: "OUT"
- board text removed: "BRWN"
- board text removed: "R5V"
- board text removed: "RNS DIODE PCB"
- board text removed: "SCAP"
- board text removed: "USB"
