File: rose/controlledWallSocket-rounded-nyoHoles.kicad_sch (KiCad schematic)
At the start: 93 parts, among them J1 screw term. 2x1 5mm, J10 IDC 6x2, J11 IDC 2x2, J12 IDC 2x2, J13 pinHeader 7x1 2.54mm, J14 pinHeader 4x1 2.54mm, J15 Conn_01x08_Pin, J2 screw term. 2x1 5mm, J3 USB_TypeC, J4 sdCard_DM3AT-SF-PEJM5, J5 IDC 2x2, J6 IDC 2x2, J7 IDC 2x2, J8 IDC 6x2, J9 IDC 2x2, M1 RTC and EEPROM, Q1 bc337, Q2 BSS138, Q3 BSS138, Q4 bc337, SW1 SW_Push, SW2 SW_Push, SW3 SW_Push, SW4 SW_Push, U1 LM66100Q, U2 LM66100Q, U3 LM66100Q, U4 LM66100Q, U5 USBLC6-2SC6, U6 LM66100Q, U7 TPS565242DRLR, U8 ESP32-S3-WROOM-1

Commit message: kicadedit
Parts:
- added Q5: bc337, Package_TO_SOT_THT:TO-92_HandSolder, symbol Transistor_BJT:BC337
Changed lines of the file:
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@@
+	)
+	(symbol
+		(lib_id "Transistor_BJT:BC337")
+		(at 92.71 196.85 90)
+		(unit 1)
+		(exclude_from_sim no)
+		(in_bom yes)
+		(on_board yes)
+		(dnp no)
+		(property "Reference" "Q5"
+			(at 91.44 191.77 0)
+			(effects
+				(font
+					(size 1.27 1.27)
+				)
+				(justify left)
+			)
+		)
+		(property "Value" "bc337"
+			(at 93.98 191.77 0)
+			(effects
+				(font
+					(size 1.27 1.27)
+				)
+				(justify left)
+			)
+		)
+		(property "Footprint" "Package_TO_SOT_THT:TO-92_HandSolder"
+			(at 94.615 191.77 0)
+			(effects
+				(font
+					(size 1.27 1.27)
+					(italic yes)
+				)
+				(justify left)
+				(hide yes)
+			)
+		)
+		(property "Datasheet" "https://diotec.com/tl_files/diotec/files/pdf/datasheets/bc337.pdf"
+			(at 92.71 196.85 0)
+			(effects
+				(font
+					(size 1.27 1.27)
+				)
+				(justify left)
+				(hide yes)
+			)
+		)
+		(property "Description" "0.8A Ic, 45V Vce, NPN Transistor, TO-92"
+			(at 92.71 196.85 0)
+			(effects
+				(font
+					(size 1.27 1.27)
+				)
+				(hide yes)
+			)
+		)
+		(pin "3"
+		)
+		(pin "1"
+		)
+		(pin "2"
+		)
+		(instances
+			(project "controlledWallSocket-rounded-nyoHoles"
+				(path "/5bec4bd2-4d25-4622-9a8f-0e623f732ee6"
+					(reference "Q5")
+					(unit 1)
+				)
+			)
+		)
 	)
 	(symbol
