File: Knop_guitar/Knop_guitar.kicad_pcb (KiCad board)
At the start: 2 copper layers, 225.3 x 282.9 mm, 3 parts

Commit message: knop guiater update
Parts:
- removed G*** (x3): LOGO, sumec_graphic:TITANFALL_ART
Routing:
- net (no net): track 2567.8 -> 0.00 mm, vias 30 -> 0
- removed copper zone on B.Cu, net (none)
- removed copper zone on F.Cu, net (none)
Other:
- board size 225.3 x 282.9 mm -> 222.9 x 282.9 mm
- board text removed: "FOOBAR1"
